Commit message: Amcl package configured

File: src/my_robot/urdf/my_robot.xacro (robot description, xacro)
@@ -2,4 +2,9 @@
 <robot name="my_robot" xmlns:xacro="http://www.ros.org/wiki/xacro">
 <xacro:include filename="$(find my_robot)/urdf/my_robot.gazebo" />
+ <!-- Length along X-axis, Width along Y-axis, Height along Z-axis -->
+  <xacro:property name="wheel_radius" value="0.075" />
+  <xacro:property name="wheel_track" value="0.3" />
+  <xacro:property name="wheel_base" value="0.3" />
+  <xacro:property name="wheel_width" value="0.05" />
   <material name="blue">
     <color rgba="0 0 0.8 1"/>
@@ -52,5 +57,5 @@
   </link>
   <joint type="continuous" name="left_front_wheel_hinge">
-    <origin xyz="0.125 0.15 0" rpy="0 0 0"/>
+    <origin xyz="${wheel_base/2} ${wheel_track/2} 0" rpy="0 0 0"/>
     <child link="left_front_wheel"/>
     <parent link="chassis"/>
@@ -72,5 +77,5 @@
       <origin xyz="0 0 0" rpy="0 1.5707 1.5707"/>
       <geometry>
-        <cylinder  radius="0.075" length="0.05"/>
+        <cylinder  radius="${wheel_radius}" length="${wheel_width}"/>
       </geometry>
     </collision>
@@ -78,5 +83,5 @@
        <origin xyz="0 0 0" rpy="0 1.5707 1.5707"/>
       <geometry>
-        <cylinder  radius="0.075" length="0.05"/>
+         <cylinder  radius="${wheel_radius}" length="${wheel_width}"/>
       </geometry>
       <material name="blue"/>
@@ -84,5 +89,5 @@
   </link>
   <joint type="continuous" name="left_rear_wheel_hinge">
-    <origin xyz="-0.125 0.15 0" rpy="0 0 0"/>
+    <origin xyz="-${wheel_base/2} ${wheel_track/2} 0" rpy="0 0 0"/>
     <child link="left_rear_wheel"/>
     <parent link="chassis"/>
@@ -104,5 +109,5 @@
       <origin xyz="0 0 0" rpy="0 1.5707 1.5707"/>
       <geometry>
-        <cylinder  radius="0.075" length="0.05"/>
+         <cylinder  radius="${wheel_radius}" length="${wheel_width}"/>
       </geometry>
     </collision>
@@ -110,5 +115,5 @@
        <origin xyz="0 0 0" rpy="0 1.5707 1.5707"/>
       <geometry>
-        <cylinder  radius="0.075" length="0.05"/>
+         <cylinder  radius="${wheel_radius}" length="${wheel_width}"/>
       </geometry>
       <material name="blue"/>
@@ -116,5 +121,5 @@
   </link>
  <joint type="continuous" name="right_front_wheel_hinge">
-    <origin xyz="0.125 -0.15 0" rpy="0 0 0"/>
+    <origin xyz="${wheel_base/2} -${wheel_track/2} 00" rpy="0 0 0"/>
     <child link="right_front_wheel"/>
     <parent link="chassis"/>
@@ -136,5 +141,5 @@
       <origin xyz="0 0 0" rpy="0 1.5707 1.5707"/>
       <geometry>
-        <cylinder  radius="0.075" length="0.05"/>
+         <cylinder  radius="${wheel_radius}" length="${wheel_width}"/>
       </geometry>
     </collision>
@@ -142,5 +147,5 @@
        <origin xyz="0 0 0" rpy="0 1.5707 1.5707"/>
       <geometry>
-        <cylinder  radius="0.075" length="0.05"/>
+         <cylinder  radius="${wheel_radius}" length="${wheel_width}"/>
       </geometry>
       <material name="blue"/>
@@ -148,5 +153,5 @@
   </link>
  <joint type="continuous" name="right_rear_wheel_hinge">
-    <origin xyz="-0.125 -0.15 0" rpy="0 0 0"/>
+    <origin xyz="-${wheel_base/2} -${wheel_track/2} 0" rpy="0 0 0"/>
     <child link="right_rear_wheel"/>
     <parent link="chassis"/>
@@ -168,5 +173,5 @@
       <origin xyz="0 0 0" rpy="0 1.5707 1.5707"/>
       <geometry>
-        <cylinder  radius="0.075" length="0.05"/>
+         <cylinder  radius="${wheel_radius}" length="${wheel_width}"/>
       </geometry>
     </collision>
@@ -174,5 +179,5 @@
        <origin xyz="0 0 0" rpy="0 1.5707 1.5707"/>
       <geometry>
-        <cylinder  radius="0.075" length="0.05"/>
+         <cylinder  radius="${wheel_radius}" length="${wheel_width}"/>
       </geometry>
       <material name="blue"/>

Commit message: adding RGB-d camera

File: src/my_robot/urdf/my_robot.xacro (robot description, xacro)
@@ -186,9 +186,9 @@
  <joint type="fixed" name="camera_joint">
     <origin xyz="0.2 0 0" rpy="0 0 0"/>
-    <child link="camera"/>
-    <parent link="chassis"/>
-    <axis xyz="0 1 0" rpy="0 0 0"/>
-  </joint>
-  <link name="camera">
+    <child link="camera_link"/>
+    <parent link="chassis"/>
+    <axis xyz="0 1 0" rpy="0 0 0"/>
+  </joint>
+  <link name="camera_link">
      <inertial>
       <mass value="0.1"/>
@@ -243,3 +243,11 @@
     </visual>
   </link>
+  <!-- Kinect camera for RTAB-Map -->
+  <joint name="camera_optical_joint" type="fixed">
+    <origin xyz="0 0 0" rpy="-1.5707 0 -1.5707"/>
+    <parent link="camera_link"/>
+    <child link="camera_link_optical"/>
+  </joint>
+  <link name="camera_link_optical">
+  </link>
 </robot>
